File: R2Fan/R2Fan.kicad_pcb (KiCad board)
At the start: 2 copper layers, 40 x 70 mm, 23 parts, among them IC2 TLP2361_V4,E, J1 XA6_SPI_Sensor, J2 XA3_Fan, J3 XT60_Power, J4 XA2_Thermister, J5 XT60_Peltier, Q1 TK40E06N1, U1 TLP250, U2 NUCLEO-G431KB

Commit message: 発注用
Connections:
- net Net-(J5-Pin_1) renamed /Plt-
Routing:
- net GND: track 0.00 -> 4.14 mm, vias 16 -> 17
- net Net-(IC2-VO_(OUTPUT)): track 6.91 -> 10.3 mm, vias 1 -> 0
- net GND2: track 53.6 -> 55.2 mm, vias 21 -> 19
- net /Plt-: vias 1 -> 59
- net (no net): vias 58 -> 0
- added copper zone on B.Cu, net /Plt-
- added copper zone on F.Cu, net /Plt-

Commit message: order ver on 20240301
Parts:
- moved C1 1.80 mm to (65.8, 71.2)
- moved IC2 1.80 mm to (65.8, 76.2)
- moved J4 1.29 mm to (78.1, 66.4)
- moved J2 1.13 mm to (68.4, 66.4)
- moved C2 0.25 mm to (81.0, 99.1)
Connections:
- U1 pad 7: Net-(R3-Pad1) -> unconnected-(U1-VO-Pad7)
Routing:
- net GND2: track 55.2 -> 57.5 mm, vias 19 -> 25
- net Net-(IC2-ANODE): track 5.45 -> 7.26 mm
- net NTC-: track 29.5 -> 28.1 mm
- net NTC+: track 26.3 -> 27.5 mm
- net Net-(IC2-VO_(OUTPUT)): track 10.3 -> 9.50 mm
