File: R2Fan/R2Fan.kicad_sch (KiCad schematic)
At the start: 18 parts, among them IC2 TLP2361_V4,E, J1 XA6_SPI_Sensor, J2 XA3_Fan, J3 XT60_Power, J4 XA2_Thermister, J5 XT60_Peltier, Q1 Q_NMOS_Depletion_GDS, U1 TLP250, U2 NUCLEO-G431KB

Commit message: for Hirayama Check
Parts:
- removed Q1: Q_NMOS_Depletion_GDS, symbol Device:Q_NMOS_Depletion_GDS
- removed TH1: Thermistor_NTC, symbol Device:Thermistor_NTC
- added Q1: TK40E06N1, Package_TO_SOT_THT:TO-220-3_Horizontal_TabDown, symbol SamacSys_Parts:TK40E06N1
- added R7: 1k, Resistor_SMD:R_0603_1608Metric, symbol Device:R
- C1, C2: footprint (none) -> Capacitor_SMD:C_0603_1608Metric
- IC2: footprint 11-4L1S(5-PIN-SOIC) -> Package_SO:MFSOP6-5_4.4x3.6mm_P1.27mm
- J1: footprint (none) -> Connector_JST:JST_XA_S06B-XASK-1_1x06_P2.50mm_Horizontal
- J2: footprint (none) -> Connector_JST:JST_XA_S03B-XASK-1_1x03_P2.50mm_Horizontal
- J3: footprint (none) -> Connector_AMASS:AMASS_XT60PW-M_1x02_P7.20mm_Horizontal
- J4: footprint (none) -> Connector_JST:JST_XA_S02B-XASK-1_1x02_P2.50mm_Horizontal
- J5: footprint (none) -> Connector_AMASS:AMASS_XT60PW-F_1x02_P7.20mm_Horizontal
- R1, R2: footprint (none) -> Resistor_SMD:R_0603_1608Metric
- R3: value 120 -> 100; footprint (none) -> Resistor_SMD:R_0603_1608Metric
- R4, R5, R6: value R -> 1k; footprint (none) -> Resistor_SMD:R_0603_1608Metric
- U2: footprint NUCLEO-G431KB:MODULE_NUCLEO-G431KB -> Tsemi2023:MODULE_NUCLEO-G431KBT6; MANUFACTURER (none) -> ST Microelectronics; PARTREV (none) -> 3; STANDARD (none) -> Manufacturer rEcommendation
Connections:
- net PA6 is gone; now on net Plt_PWM: R2.1
- net +3.3V: now also R6.1
- net Fan_PWM: now also U2.3_2 (PA10); no longer U2.4_9 (PA4)
- net GND: now also R5.2, R7.2; no longer R6.2
- net GND2: now also J3.1 (Pin_1), Q1.3; no longer J3.2 (Pin_2)
- net NTC+: now also J4.2 (Pin_2), R4.2, R6.2; no longer J4.1 (Pin_1)
- net NTC-: now also J4.1 (Pin_1), R5.1, R7.1; no longer J4.2 (Pin_2)
- net Vdrive: now also C2.1, J3.2 (Pin_2), U1.8 (VCC); no longer J3.1 (Pin_1)
- net at R3.2: now also Q1.1
- net at J5.1 (Pin_1): now also Q1.2
- removed net ADC+: R4.2, R5.1
- removed net ADC-: R5.2, R6.1
Other:
- moved on the sheet: J1, J4, R4, U2A, U2B

Commit message: 発注用
Connections:
- net Plt-: now reaches J5.1 (Pin_1), Q1.2
- no-connect marks 0 -> 19

Commit message: order ver on 20240301
Connections:
- net at R3.1, U1.6 (VO): no longer U1.7 (VO)
- no-connect marks 19 -> 20
